File: ForgetMeNot_v2/ForgetMeNot_v2.kicad_sch (KiCad schematic)
At the start: 44 parts, among them J1 Conn_01x04, SW1 SW_Push, U1 RP2040, U2 W25Q128JVS, U3 NCP1117, U4 LIS2HH12, U5 MCP1640x-xMC, Y1 Crystal_ABM8

Commit message: finished layout & tracing
Parts:
- added C22: 100n, Capacitor_SMD:C_0402_1005Metric, symbol Device:C
- SW1: footprint Button_Switch_SMD:SW_Push_1TS009xxxx-xxxx-xxxx_6x6x5mm -> Button_Switch_SMD:SW_SPST_PTS647_Sx38
- TP1: footprint TestPoint:TestPoint_THTPad_1.5x1.5mm_Drill0.7mm -> TestPoint:TestPoint_THTPad_1.0x1.0mm_Drill0.5mm
- TP2: footprint TestPoint:TestPoint_THTPad_1.5x1.5mm_Drill0.7mm -> TestPoint:TestPoint_THTPad_D1.0mm_Drill0.5mm
Connections:
- net +3.3V: now also C22.1
- net ACC_CS: now also U1.29 (GPIO18); no longer U1.34 (GPIO22)
- net ACC_INT: now also U1.31 (GPIO20); no longer U1.36 (GPIO24)
- net ACC_SCL: now also U1.30 (GPIO19); no longer U1.35 (GPIO23)
- net ACC_SDA: now also U1.27 (GPIO16); no longer U1.31 (GPIO20)
- net ACC_SDO: now also U1.28 (GPIO17); no longer U1.32 (GPIO21)
- net BUZZ: now also U1.32 (GPIO21); no longer U1.29 (GPIO18)
- net GND: now also C22.2
- net LED: now also U1.2 (GPIO0); no longer U1.14 (GPIO11)
- net ZERO: now also U1.34 (GPIO22); no longer U1.30 (GPIO19)
Other:
- moved on the sheet: C17, C18, C19, U4
